Commit message: fixed spawning drone in gazebo. Now the drone spawns properly

File: falco_ws/src/drone/urdf/quadrotor_base.urdf.xacro (robot description, xacro)
@@ -13,5 +13,5 @@
         <origin xyz="0 0 0" rpy="0 0 0" />
         <geometry>
-          <mesh filename="package://imav_2017/meshes/quadrotor/quadrotor_4.dae"/>
+          <mesh filename="file:///github/falco_ws/src/drone/meshes/quadrotor/quadrotor_base.dae"/>
         </geometry>
       </visual>
@@ -19,5 +19,5 @@
         <origin xyz="0 0 0" rpy="0 0 0" />
         <geometry>
-          <mesh filename="package://imav_2017/meshes/quadrotor/quadrotor_4.stl"/>
+          <mesh filename="file:///github/falco_ws/src//drone/meshes/quadrotor/quadrotor_base.stl"/>
         </geometry>
       </collision>

File: falco_ws/src/drone/urdf/qws.urdf (robot description, URDF)
Before this commit: robot quadrotor_full, 3 links, 2 joints
Links:
- link base_link: geometry collision mesh filename=file:///github/falco_ws/src//drone/meshes/quadrotor/quadrot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; visual mesh filename=file:///github/falco_ws/src/drone/meshes/quadrotor/quadroto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

File: falco_ws/src/drone/urdf/sensors/hokuyo_utm30lx.urdf.xacro (robot description, xacro)
@@ -16,5 +16,5 @@
 	  <origin xyz="0 0 0" rpy="0 0 0" />
           <geometry>
-          <mesh filename="package://imav_2017/meshes/hokuyo_utm30lx/hokuyo_utm_30lx$(optenv TEST_SELF_FILTER).dae"/>
+          <mesh filename="file:///github/falco_ws/src/meshes/hokuyo_utm30lx/hokuyo_utm_30lx$(optenv TEST_SELF_FILTER).dae"/>
         </geometry>
 	</visual>
@@ -23,5 +23,5 @@
           <geometry>
           <box size="0.058 0.058 0.087" />
-          <mesh filename="package://hector_sensors_description/meshes/hokuyo_utm30lx/hokuyo_utm_30lx.stl"/>
+          <mesh filename="file:///github/falco_ws/src/meshes/hokuyo_utm30lx/hokuyo_utm_30lx.stl"/>
         </geometry>
 	</collision>

File: falco_ws/src/drone/urdf/sensors/sonar_sensor.urdf.xacro (robot description, xacro)
@@ -17,5 +17,5 @@
         <geometry>
           <!--<box size="0.01 0.01 0.01" /> -->
-          <mesh filename="package://imav_2017/meshes/sonar_sensor/max_sonar_ez4.dae"/>
+          <mesh filename="file:///github/falco_ws/src/meshes/sonar_sensor/max_sonar_ez4.dae"/>
         </geometry>
       </visual>
