Commit message: added ros2_control interface for gazebo

File: falco_ws/src/drone/urdf/FALCO.urdf.xacro (robot description, xacro)
@@ -1,5019 +1,5081 @@
 <?xml version='1.0' encoding='utf-8'?>
 <robot name="FALCO">
-    <link name="FALCO_Piastra_Inferiore_newBOZZA">
-        <inertial>
-            <origin xyz="0.0 0.0 0.0" rpy="0.0 0.0 0.0" />
-            <mass value="0.0" />
-            <inertia ixx="0.0" iyy="0.0" izz="0.0" ixy="0.0" iyz="0.0" ixz="0.0" />
-        </inertial>
-        <visual name="FALCO_Piastra_Inferiore_newBOZZA_visual">
-            <origin xyz="0.0 0.0 0.0" rpy="0.0 0.0 0.0" />
+    <xacro:macro name="quadrotor_macro">
+        <link name="FALCO_Piastra_Inferiore_newBOZZA">
+            <inertial>
+                <origin xyz="0.0 0.0 0.0" rpy="0.0 0.0 0.0" />
+                <mass value="0.0" />
+                <inertia ixx="0.0" iyy="0.0" izz="0.0" ixy="0.0" iyz="0.0" ixz="0.0" />
+            </inertial>
+            <visual name="FALCO_Piastra_Inferiore_newBOZZA_visual">
+                <origin xyz="0.0 0.0 0.0" rpy="0.0 0.0 0.0" />
+                <geometry>
+                    <mesh filename="meshes/FALCO_Piastra_Inferiore_newBOZZA.stl" scale="0.001 0.001 0.001" />
+                </geometry>
+            </visual>
+            <collision name="FALCO_Piastra_Inferiore_newBOZZA_collision">
+                <origin xyz="0.0 0.0 0.0" rpy="0.0 0.0 0.0" />
+                <geometry>
+                    <mesh filename="meshes/FALCO_Piastra_Inferiore_newBOZZA.stl" scale="0.001 0.001 0.001" />
+                </geometry>
+            </collision>
+        </link>
+        <link name="FALCO_Base-plate-BOZZA_8">
+            <inertial>
+                <origin xyz="-0.0643272897434528 0.0030000000000000005 0.011313708499999799" rpy="0.0 0.0 0.0" />
+                <mass value="0.0" />
+                <inertia ixx="0.0" iyy="0.0" izz="0.0" ixy="0.0" iyz="0.0" ixz="0.0" />
+            </inertial>
+            <visual name="FALCO_Base-plate-BOZZA_visual">
+                <origin xyz="0.0 0.0 0.0" rpy="0.0 0.0 0.0" />
+                <geometry>
+                    <mesh filename="meshes/FALCO_Base-plate-BOZZA.stl" scale="0.001 0.001 0.001" />
+                </geometry>
+            </visual>
+            <collision name="FALCO_Base-plate-BOZZA_collision">
+                <origin xyz="0.0 0.0 0.0" rpy="0.0 0.0 0.0" />
+                <geometry>
+                    <mesh filename="meshes/FALCO_Base-plate-BOZZA.stl" scale="0.001 0.001 0.001" />
+                </geometry>
+            </collision>
+        </link>
+        <link name="FALCO_Holder-BOZZA_32">
+            <inertial>
+                <origin xyz="0.0067562915000006505 -0.0174999999999982 0.11692728974345301" rpy="0.0 0.0 0.0" />
+                <mass value="0.0" />
+                <inertia ixx="0.0" iyy="0.0" izz="0.0" ixy="0.0" iyz="0.0" ixz="0.0" />
+            </inertial>
+            <visual name="FALCO_Holder-BOZZA_visual">
+                <origin xyz="0.0 0.0 0.0" rpy="0.0 0.0 0.0" />
+                <geometry>
+                    <mesh filename="meshes/FALCO_Holder-BOZZA.stl" scale="0.001 0.001 0.001" />
+                </geometry>
+            </visual>
+            <collision name="FALCO_Holder-BOZZA_collision">
+                <origin xyz="0.0 0.0 0.0" rpy="0.0 0.0 0.0" />
+                <geometry>
+                    <mesh filename="meshes/FALCO_Holder-BOZZA.stl" scale="0.001 0.001 0.001" />
+                </geometry>
+            </collision>
+        </link>
+        <link name="FALCO_Arm-BOZZA_4">
+            <inertial>
+                <origin xyz="-0.244177289743444 -0.017126035512196595 -0.003598464563865124" rpy="0.0 0.0 0.0" />
+                <mass value="0.0" />
+                <inertia ixx="0.0" iyy="0.0" izz="0.0" ixy="0.0" iyz="0.0" ixz="0.0" />
+            </inertial>
+            <visual name="FALCO_Arm-BOZZA_visual">
+                <origin xyz="0.0 0.0 0.0" rpy="0.0 0.0 0.0" />
+                <geometry>
+                    <mesh filename="meshes/FALCO_Arm-BOZZA.stl" scale="0.001 0.001 0.001" />
+                </geometry>
+            </visual>
+            <collision name="FALCO_Arm-BOZZA_collision">
+                <origin xyz="0.0 0.0 0.0" rpy="0.0 0.0 0.0" />
+                <geometry>
+                    <mesh filename="meshes/FALCO_Arm-BOZZA.stl" scale="0.001 0.001 0.001" />
+                </geometry>
+            </collision>
+        </link>
+        <link name="FALCO_Plate-motor-BOZZA_4">
+            <inertial>
+                <origin xyz="6.29149998127021e-06 -0.0317499999999791 0.346427289743446" rpy="0.0 0.0 0.0" />
+                <mass value="0.0" />
+                <inertia ixx="0.0" iyy="0.0" izz="0.0" ixy="0.0" iyz="0.0" ixz="0.0" />
+            </inertial>
+            <visual name="FALCO_Plate-motor-BOZZA_visual">
+                <origin xyz="0.0 0.0 0.0" rpy="0.0 0.0 0.0" />
+                <geometry>
+                    <mesh filename="meshes/FALCO_Plate-motor-BOZZA.stl" scale="0.001 0.001 0.001" />
+                </geometry>
+            </visual>
+            <collision name="FALCO_Plate-motor-BOZZA_collision">
+                <origin xyz="0.0 0.0 0.0" rpy="0.0 0.0 0.0" />
+                <geometry>
+                    <mesh filename="meshes/FALCO_Plate-motor-BOZZA.stl" scale="0.001 0.001 0.001" />
+                </geometry>
+            </collision>
+        </link>
+        <link name="FALCO_Spessore-BOZZA_4">
+            <inertial>
+                <origin xyz="6.298841940227671e-06 -0.0339999999999791 0.346427297085394" rpy="0.0 0.0 0.0" />
+                <mass value="0.0" />
+                <inertia ixx="0.0" iyy="0.0" izz="0.0" ixy="0.0" iyz="0.0" ixz="0.0" />
+            </inertial>
+            <visual name="FALCO_Spessore-BOZZA_visual">
+                <origin xyz="0.0 0.0 0.0" rpy="0.0 0.0 0.0" />
+                <geometry>
+                    <mesh filename="meshes/FALCO_Spessore-BOZZA.stl" scale="0.001 0.001 0.001" />
+                </geometry>
+            </visual>
+            <collision name="FALCO_Spessore-BOZZA_collision">
+                <origin xyz="0.0 0.0 0.0" rpy="0.0 0.0 0.0" />
+                <geometry>
+                    <mesh filename="meshes/FALCO_Spessore-BOZZA.stl" scale="0.001 0.001 0.001" />
+                </geometry>
+            </collision>
+        </link>
+        <link name="FALCO_Arm-plate-BOZZA_8">
+            <inertial>
+                <origin xyz="0.137927289743454 0.032999999999998204 -0.014743708499999402" rpy="0.0 0.0 0.0" />
+                <mass value="0.0" />
+                <inertia ixx="0.0" iyy="0.0" izz="0.0" ixy="0.0" iyz="0.0" ixz="0.0" />
+            </inertial>
+            <visual name="FALCO_Arm-plate-BOZZA_visual">
+                <origin xyz="0.0 0.0 0.0" rpy="0.0 0.0 0.0" />
+                <geometry>
+                    <mesh filename="meshes/FALCO_Arm-plate-BOZZA.stl" scale="0.001 0.001 0.001" />
+                </geometry>
+            </visual>
+            <collision name="FALCO_Arm-plate-BOZZA_collision">
+                <origin xyz="0.0 0.0 0.0" rpy="0.0 0.0 0.0" />
+                <geometry>
+                    <mesh filename="meshes/FALCO_Arm-plate-BOZZA.stl" scale="0.001 0.001 0.001" />
+                </geometry>
+            </collision>
+        </link>
+        <link name="FALCO_Big-pin-BOZZA_8">
+            <inertial>
+                <origin xyz="6.291500000726871e-06 -0.0169999999999802 0.10532728974345501" rpy="0.0 0.0 0.0" />
+                <mass value="0.0" />
+                <inertia ixx="0.0" iyy="0.0" izz="0.0" ixy="0.0" iyz="0.0" ixz="0.0" />
+            </inertial>
+            <visual name="FALCO_Big-pin-BOZZA_visual">
+                <origin xyz="0.0 0.0 0.0" rpy="0.0 0.0 0.0" />
+                <geometry>
+                    <mesh filename="meshes/FALCO_Big-pin-BOZZA.stl" scale="0.001 0.001 0.001" />
+                </geometry>
+            </visual>
+            <collision name="FALCO_Big-pin-BOZZA_collision">
+                <origin xyz="0.0 0.0 0.0" rpy="0.0 0.0 0.0" />
+                <geometry>
+                    <mesh filename="meshes/FALCO_Big-pin-BOZZA.stl" scale="0.001 0.001 0.001" />
+                </geometry>
+            </collision>
+        </link>
+        <link name="FALCO_Pin-BOZZA_4">
+            <inertial>
+                <origin xyz="6.291500000699111e-06 -0.026999999999980206 0.10532728974345702" rpy="0.0 0.0 0.0" />
+                <mass value="0.0" />
+                <inertia ixx="0.0" iyy="0.0" izz="0.0" ixy="0.0" iyz="0.0" ixz="0.0" />
+            </inertial>
+            <visual name="FALCO_Pin-BOZZA_visual">
+                <origin xyz="0.0 0.0 0.0" rpy="0.0 0.0 0.0" />
+                <geometry>
+                    <mesh filename="meshes/FALCO_Pin-BOZZA.stl" scale="0.001 0.001 0.001" />
+                </geometry>
+            </visual>
+            <collision name="FALCO_Pin-BOZZA_collision">
+                <origin xyz="0.0 0.0 0.0" rpy="0.0 0.0 0.0" />
+                <geometry>
+                    <mesh filename="meshes/FALCO_Pin-BOZZA.stl" scale="0.001 0.001 0.001" />
+                </geometry>
+            </collision>
+        </link>
+        <link name="FALCO_plain-washer-clevis-pin-grade-a_iso_ISO-8738---3_16">
+            <inertial>
+                <origin xyz="0.0010000000000229502 -0.0752647612219163 0.36393660795731125" rpy="0.0 0.0 0.0" />
+                <mass value="0.0" />
+                <inertia ixx="0.0" iyy="0.0" izz="0.0" ixy="0.0" iyz="0.0" ixz="0.0" />
+            </inertial>
+            <visual name="FALCO_plain-washer-clevis-pin-grade-a_iso_ISO-8738---3_visual">
+                <origin xyz="0.0 0.0 0.0" rpy="0.0 0.0 0.0" />
+                <geometry>
+                    <mesh filename="meshes/FALCO_plain-washer-clevis-pin-grade-a_iso_ISO-8738---3.stl" scale="0.001 0.001 0.001" />
+                </geometry>
+            </visual>
+            <collision name="FALCO_plain-washer-clevis-pin-grade-a_iso_ISO-8738---3_collision">
+                <origin xyz="0.0 0.0 0.0" rpy="0.0 0.0 0.0" />
+                <geometry>
+                    <mesh filename="meshes/FALCO_plain-washer-clevis-pin-grade-a_iso_ISO-8738---3.stl" scale="0.001 0.001 0.001" />
+                </geometry>
+            </collision>
+        </link>
+        <link name="FALCO_torque-nut-01_iso_ISO-7040-M3-N_32">
+            <inertial>
+                <origin xyz="0.13492728974345702 -0.029999999999974603 -0.018156291500000598" rpy="0.0 0.0 0.0" />
+                <mass value="0.0" />
+                <inertia ixx="0.0" iyy="0.0" izz="0.0" ixy="0.0" iyz="0.0" ixz="0.0" />
+            </inertial>
+            <visual name="FALCO_torque-nut-01_iso_ISO-7040-M3-N_visual">
+                <origin xyz="0.0 0.0 0.0" rpy="0.0 0.0 0.0" />
+                <geometry>
+                    <mesh filename="meshes/FALCO_torque-nut-01_iso_ISO-7040-M3-N.stl" scale="0.001 0.001 0.001" />
+                </geometry>
+            </visual>
+            <collision name="FALCO_torque-nut-01_iso_ISO-7040-M3-N_collision">
+                <origin xyz="0.0 0.0 0.0" rpy="0.0 0.0 0.0" />
+                <geometry>
+                    <mesh filename="meshes/FALCO_torque-nut-01_iso_ISO-7040-M3-N.stl" scale="0.001 0.001 0.001" />
+                </geometry>
+            </collision>
+        </link>
+        <link name="FALCO_socket-head-cap-screw_iso_ISO-4762-M2.5-x-8---8N_16">
+            <inertial>
+                <origin xyz="-0.028499999999979 -0.0710284539218816 0.33929815562436977" rpy="0.0 0.0 0.0" />
+                <mass value="0.0" />
+                <inertia ixx="0.0" iyy="0.0" izz="0.0" ixy="0.0" iyz="0.0" ixz="0.0" />
+            </inertial>
+            <visual name="FALCO_socket-head-cap-screw_iso_ISO-4762-M2.5-x-8---8N_visual">
+                <origin xyz="0.0 0.0 0.0" rpy="0.0 0.0 0.0" />
+                <geometry>
+                    <mesh filename="meshes/FALCO_socket-head-cap-screw_iso_ISO-4762-M2.5-x-8---8N.stl" scale="0.001 0.001 0.001" />
+                </geometry>
+            </visual>
+            <collision name="FALCO_socket-head-cap-screw_iso_ISO-4762-M2.5-x-8---8N_collision">
+                <origin xyz="0.0 0.0 0.0" rpy="0.0 0.0 0.0" />
+                <geometry>
+                    <mesh filename="meshes/FALCO_socket-head-cap-screw_iso_ISO-4762-M2.5-x-8---8N.stl" scale="0.001 0.001 0.001" />
+                </geometry>
+            </collision>
+        </link>
+        <link name="FALCO_socket-head-cap-screw_am_B18.3.1M---3-x-0.5-x-35-Hex-SHCS----18NHX_32">
+            <inertial>
+                <origin xyz="0.0048000000000189506 -0.042153671337499 0.31889600708802796" rpy="0.0 0.0 0.0" />
+                <mass value="0.0" />
+                <inertia ixx="0.0" iyy="0.0" izz="0.0" ixy="0.0" iyz="0.0" ixz="0.0" />
+            </inertial>
+            <visual name="FALCO_socket-head-cap-screw_am_B18.3.1M---3-x-0.5-x-35-Hex-SHCS----18NHX_visual">
+                <origin xyz="0.0 0.0 0.0" rpy="0.0 0.0 0.0" />
+                <geometry>
+                    <mesh filename="meshes/FALCO_socket-head-cap-screw_am_B18.3.1M---3-x-0.5-x-35-Hex-SHCS----18NHX.stl" scale="0.001 0.001 0.001" />
+                </geometry>
+            </visual>
+            <collision name="FALCO_socket-head-cap-screw_am_B18.3.1M---3-x-0.5-x-35-Hex-SHCS----18NHX_collision">
+                <origin xyz="0.0 0.0 0.0" rpy="0.0 0.0 0.0" />
+                <geometry>
+                    <mesh filename="meshes/FALCO_socket-head-cap-screw_am_B18.3.1M---3-x-0.5-x-35-Hex-SHCS----18NHX.stl" scale="0.001 0.001 0.001" />
+                </geometry>
+            </collision>
+        </link>
+        <link name="FALCO_outer.step_4">
+            <inertial>
+                <origin xyz="6.298842000679321e-06 -0.34642729708541703 -0.035499999999979104" rpy="0.0 0.0 0.0" />
+                <mass value="0.0" />
+                <inertia ixx="0.0" iyy="0.0" izz="0.0" ixy="0.0" iyz="0.0" ixz="0.0" />
+            </inertial>
+            <visual name="FALCO_outer.step_visual">
+                <origin xyz="0.0 0.0 0.0" rpy="0.0 0.0 0.0" />
+                <geometry>
+                    <mesh filename="meshes/FALCO_outer.step.stl" scale="0.001 0.001 0.001" />
+                </geometry>
+            </visual>
+            <collision name="FALCO_outer.step_collision">
+                <origin xyz="0.0 0.0 0.0" rpy="0.0 0.0 0.0" />
+                <geometry>
+                    <mesh filename="meshes/FALCO_outer.step.stl" scale="0.001 0.001 0.001" />
+                </geometry>
+            </collision>
+        </link>
+        <link name="FALCO_inner.step_4">
+            <inertial>
+                <origin xyz="6.298842000679321e-06 -0.34642729708541703 -0.035499999999979104" rpy="0.0 0.0 0.0" />
+                <mass value="0.0" />
+                <inertia ixx="0.0" iyy="0.0" izz="0.0" ixy="0.0" iyz="0.0" ixz="0.0" />
+            </inertial>
+            <visual name="FALCO_inner.step_visual">
+                <origin xyz="0.0 0.0 0.0" rpy="0.0 0.0 0.0" />
+                <geometry>
+                    <mesh filename="meshes/FALCO_inner.step.stl" scale="0.001 0.001 0.001" />
+                </geometry>
+            </visual>
+            <collision name="FALCO_inner.step_collision">
+                <origin xyz="0.0 0.0 0.0" rpy="0.0 0.0 0.0" />
+                <geometry>
+                    <mesh filename="meshes/FALCO_inner.step.stl" scale="0.001 0.001 0.001" />
+                </geometry>
+            </collision>
+        </link>
+        <link name="FALCO_BOTTOM.step_4">
+            <inertial>
+                <origin xyz="6.298842000679321e-06 -0.34642729708541703 -0.035499999999979104" rpy="0.0 0.0 0.0" />
+                <mass value="0.0" />
+                <inertia ixx="0.0" iyy="0.0" izz="0.0" ixy="0.0" iyz="0.0" ixz="0.0" />
+            </inertial>
+            <visual name="FALCO_BOTTOM.step_visual">
+                <origin xyz="0.0 0.0 0.0" rpy="0.0 0.0 0.0" />
+                <geometry>
+                    <mesh filename="meshes/FALCO_BOTTOM.step.stl" scale="0.001 0.001 0.001" />
+                </geometry>
+            </visual>
+            <collision name="FALCO_BOTTOM.step_collision">
+                <origin xyz="0.0 0.0 0.0" rpy="0.0 0.0 0.0" />
+                <geometry>
+                    <mesh filename="meshes/FALCO_BOTTOM.step.stl" scale="0.001 0.001 0.001" />
+                </geometry>
+            </collision>
+        </link>
+        <link name="FALCO_TOP.step_4">
+            <inertial>
+                <origin xyz="6.298842000679321e-06 -0.34642729708541703 -0.035499999999979104" rpy="0.0 0.0 0.0" />
+                <mass value="0.0" />
+                <inertia ixx="0.0" iyy="0.0" izz="0.0" ixy="0.0" iyz="0.0" ixz="0.0" />
+            </inertial>
+            <visual name="FALCO_TOP.step_visual">
+                <origin xyz="0.0 0.0 0.0" rpy="0.0 0.0 0.0" />
+                <geometry>
+                    <mesh filename="meshes/FALCO_TOP.step.stl" scale="0.001 0.001 0.001" />
+                </geometry>
+            </visual>
+            <collision name="FALCO_TOP.step_collision">
+                <origin xyz="0.0 0.0 0.0" rpy="0.0 0.0 0.0" />
+                <geometry>
+                    <mesh filename="meshes/FALCO_TOP.step.stl" scale="0.001 0.001 0.001" />
+                </geometry>
+            </collision>
+        </link>
+        <link name="FALCO_shaft.step_4">
+            <inertial>
+                <origin xyz="6.298842000647e-06 -0.34642729708541403 0.00100000000002094" rpy="0.0 0.0 0.0" />
+                <mass value="0.0" />
+                <inertia ixx="0.0" iyy="0.0" izz="0.0" ixy="0.0" iyz="0.0" ixz="0.0" />
+            </inertial>
+            <visual name="FALCO_shaft.step_visual">
+                <origin xyz="0.0 0.0 0.0" rpy="0.0 0.0 0.0" />
+                <geometry>
+                    <mesh filename="meshes/FALCO_shaft.step.stl" scale="0.001 0.001 0.001" />
+                </geometry>
+            </visual>
+            <collision name="FALCO_shaft.step_collision">
+                <origin xyz="0.0 0.0 0.0" rpy="0.0 0.0 0.0" />
+                <geometry>
+                    <mesh filename="meshes/FALCO_shaft.step.stl" scale="0.001 0.001 0.001" />
+                </geometry>
+            </collision>
+        </link>
+        <link name="FALCO_clip.step_4">
+            <inertial>
+                <origin xyz="6.298842000679321e-06 -0.34642729708541703 -0.035499999999979104" rpy="0.0 0.0 0.0" />
+                <mass value="0.0" />
+                <inertia ixx="0.0" iyy="0.0" izz="0.0" ixy="0.0" iyz="0.0" ixz="0.0" />
+            </inertial>
+            <visual name="FALCO_clip.step_visual">
+                <origin xyz="0.0 0.0 0.0" rpy="0.0 0.0 0.0" />
+                <geometry>
+                    <mesh filename="meshes/FALCO_clip.step.stl" scale="0.001 0.001 0.001" />
+                </geometry>
+            </visual>
+            <collision name="FALCO_clip.step_collision">
+                <origin xyz="0.0 0.0 0.0" rpy="0.0 0.0 0.0" />
+                <geometry>
+                    <mesh filename="meshes/FALCO_clip.step.stl" scale="0.001 0.001 0.001" />
+                </geometry>
+            </collision>
+        </link>
+        <link name="FALCO_Elica-bozza-v3SpecchioSpecchio.step_4">
+            <inertial>
+                <origin xyz="0.27790102034813613 0.2068402646852157 -0.07149999999997761" rpy="0.0 0.0 0.0" />
+                <mass value="0.0" />
+                <inertia ixx="0.0" iyy="0.0" izz="0.0" ixy="0.0" iyz="0.0" ixz="0.0" />
+            </inertial>
+            <visual name="FALCO_Elica-bozza-v3SpecchioSpecchio.step_visual">
+                <origin xyz="0.0 0.0 0.0" rpy="0.0 0.0 0.0" />
+                <geometry>
+                    <mesh filename="meshes/FALCO_Elica-bozza-v3SpecchioSpecchio.step.stl" scale="0.001 0.001 0.001" />
+                </geometry>
+            </visual>
+            <collision name="FALCO_Elica-bozza-v3SpecchioSpecchio.step_collision">
+                <origin xyz="0.0 0.0 0.0" rpy="0.0 0.0 0.0" />
+                <geometry>
+                    <mesh filename="meshes/FALCO_Elica-bozza-v3SpecchioSpecchio.step.stl" scale="0.001 0.001 0.001" />
+                </geometry>
+            </collision>
+        </link>
+        <link name="FALCO_Gamba_nuova_4">
+            <inertial>
+                <origin xyz="-0.346428998398863 -0.00100000000002095 -6.2915000601238e-06" rpy="0.0 0.0 0.0" />
+                <mass value="0.0" />
+                <inertia ixx="0.0" iyy="0.0" izz="0.0" ixy="0.0" iyz="0.0" ixz="0.0" />
+            </inertial>
+            <visual name="FALCO_Gamba_nuova_visual">
+                <origin xyz="0.0 0.0 0.0" rpy="0.0 0.0 0.0" />
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
File: falco_ws/src/drone/urdf/quadrotor.urdf.xacro (robot description, xacro)
@@ -1,21 +1,15 @@
 <?xml version="1.0"?>
-<robot name="quadrotor_full" xmlns:xacro="http://wiki.ros.org/xacro" >
-    <!-- Declare the 'id' argument -->
-    <xacro:arg name="id" default="0"/>
-    <!-- Use the argument -->
-    <xacro:property name="ID" value="$(arg id)" />
-    <xacro:property name="robot_name" value="quadrotor_$(arg id)" />
-    <xacro:property name="M_PI" value="3.1415926535897931" />
-    <!-- Included URDF Files -->
-    <!-- Base airframe -->
-    <xacro:include filename="$(find drone)/urdf/quadrotor_base.urdf.xacro" />
-    <xacro:quadrotor_base_macro/>
-    <!-- IMU, Baro, Magnetic, GPS, Groundtruth sensors -->
-    <xacro:include filename="$(find drone)/urdf/sensors/quadrotor_sensors.urdf.xacro" />
-    <xacro:quadrotor_sensors robot_name="${robot_name}"/>
-    <!-- Forward facing camera -->
-    <xacro:include filename="$(find drone)/urdf/sensors/generic_camera.urdf.xacro" />
-    <xacro:generic_camera name="front" robot_name="${robot_name}" parent="base_link" update_rate="60" res_x="640" res_y="360" image_format="R8G8B8" hfov="${81*M_PI/180}">
-      <origin xyz="0.21 0.0 0.01" rpy="0 0 0"/>
-    </xacro:generic_camera>
+<robot name="quadrotor_full" xmlns:xacro="http://wiki.ros.org/xacro">
+  <xacro:arg name="id" default="0"/>
+  <xacro:property name="ID" value="$(arg id)"/>
+  <xacro:property name="robot_name" value="quadrotor_$(arg id)"/>
+  <xacro:property name="M_PI" value="3.1415926535897931"/>
+  <xacro:include filename="$(find drone)/urdf/quadrotor_base.urdf.xacro"/>
+  <xacro:quadrotor_base_macro/>
+  <xacro:include filename="$(find drone)/urdf/sensors/quadrotor_sensors.urdf.xacro"/>
+  <xacro:quadrotor_sensors robot_name="${robot_name}"/>
+  <xacro:include filename="$(find drone)/urdf/sensors/generic_camera.urdf.xacro"/>
+  <xacro:generic_camera name="front" robot_name="${robot_name}" parent="base_link" update_rate="60" res_x="640" res_y="360" image_format="R8G8B8" hfov="${81*M_PI/180}">
+    <origin xyz="0.21 0.0 0.01" rpy="0 0 0"/>
+  </xacro:generic_camera>
 </robot>
