Commit message: added ros2_control interface for gazebo

File: falco_ws/src/drone/urdf/quadrotor_base.urdf.xacro (robot description, xacro)
@@ -1,15 +1,13 @@
 <?xml version="1.0"?>
-<robot xmlns:xacro="http://wiki.ros.org/xacro" >
-  <!-- Main quadrotor link -->
+<robot xmlns:xacro="http://wiki.ros.org/xacro" name="quadrotor">
   <xacro:macro name="quadrotor_base_macro">
+    <!-- Base Link -->
     <link name="base_link">
       <inertial>
-	<origin xyz="0 0 0" rpy="0 0 0" />
-        <mass value="1.477" />
-        <origin xyz="0 0 0" />
-        <inertia ixx="0.01152" ixy="0.0" ixz="0.0" iyy="0.01152" iyz="0.0" izz="0.0218" />
+        <origin xyz="0 0 0" rpy="0 0 0"/>
+        <mass value="1.477"/>
+        <inertia ixx="0.01152" ixy="0.0" ixz="0.0" iyy="0.01152" iyz="0.0" izz="0.0218"/>
       </inertial>
       <visual>
-        <origin xyz="0 0 0" rpy="0 0 0" />
         <geometry>
           <mesh filename="file:///github/falco_ws/src/drone/meshes/quadrotor/quadrotor_base.dae"/>
@@ -17,10 +15,69 @@
       </visual>
       <collision>
-        <origin xyz="0 0 0" rpy="0 0 0" />
         <geometry>
-          <mesh filename="file:///github/falco_ws/src//drone/meshes/quadrotor/quadrotor_base.stl"/>
+          <mesh filename="file:///github/falco_ws/src/drone/meshes/quadrotor/quadrotor_base.stl"/>
         </geometry>
       </collision>
     </link>
+    <!-- ROS 2 Control Configuration -->
+    <ros2_control name="GazeboSimSystem" type="system">
+      <hardware>
+        <plugin>gazebo_ros2_control/GazeboSimSystem</plugin>
+      </hardware>
+      <joint name="rotor_1_joint">
+        <command_interface name="velocity"/>
+        <state_interface name="position"/>
+        <state_interface name="velocity"/>
+      </joint>
+      <joint name="rotor_2_joint">
+        <command_interface name="velocity"/>
+        <state_interface name="position"/>
+        <state_interface name="velocity"/>
+      </joint>
+      <joint name="rotor_3_joint">
+        <command_interface name="velocity"/>
+        <state_interface name="position"/>
+        <state_interface name="velocity"/>
+      </joint>
+      <joint name="rotor_4_joint">
+        <command_interface name="velocity"/>
+        <state_interface name="position"/>
+        <state_interface name="velocity"/>
+      </joint>
+    </ros2_control>
+    <!-- Rotor Macro -->
+    <xacro:macro name="rotor" params="prefix x y">
+      <joint name="${prefix}_joint" type="continuous">
+        <parent link="base_link"/>
+        <child link="${prefix}_link"/>
+        <origin xyz="${x} ${y} 0.1" rpy="0 0 0"/>
+        <axis xyz="0 0 1"/>
+      </joint>
+      <link name="${prefix}_link">
+        <inertial>
+          <mass value="0.1"/>
+          <inertia ixx="0.0001" ixy="0" ixz="0" iyy="0.0001" iyz="0" izz="0.0002"/>
+        </inertial>
+        <visual>
+          <geometry>
+            <cylinder length="0.02" radius="0.1"/>
+          </geometry>
+        </visual>
+      </link>
+    </xacro:macro>
+    <!-- Create 4 rotors -->
+    <xacro:rotor prefix="rotor_1" x="0.2" y="0.2"/>
+    <xacro:rotor prefix="rotor_2" x="-0.2" y="0.2"/>
+    <xacro:rotor prefix="rotor_3" x="-0.2" y="-0.2"/>
+    <xacro:rotor prefix="rotor_4" x="0.2" y="-0.2"/>
+    <!-- ROS 2 Gazebo Plugin -->
+    <gazebo>
+      <plugin name="gazebo_ros2_control" filename="libgazebo_ros2_control.so">
+        <robotNamespace>/</robotNamespace>
+        <robot_param>robot_description</robot_param>
+      </plugin>
+    </gazebo>
   </xacro:macro>
+  <!-- Instantiate macro -->
+  <xacro:quadrotor_base_macro/>
 </robot>

File: falco_ws/src/drone/urdf/qws.urdf (robot description, URDF)
Before this commit: robot quadrotor_full, 3 links, 2 joints
Links:
- added link rotor_1_link, mass 0.1; visual cylinder length=0.02 radius=0.1
- added link rotor_2_link, mass 0.1; visual cylinder length=0.02 radius=0.1
- added link rotor_3_link, mass 0.1; visual cylinder length=0.02 radius=0.1
- added link rotor_4_link, mass 0.1; visual cylinder length=0.02 radius=0.1
- link base_link: geometry collision mesh filename=file:///github/falco_ws/src/drone/meshes/quadrotor/quadroto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; visual mesh filename=file:///github/falco_ws/src/drone/meshes/quadrotor/quadroto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
Joints:
- added joint rotor_1_joint: type continuous, parent base_link, child rotor_1_link, origin xyz=0.2 0.2 0.1 rpy=0 0 0, axis 0 0 1
- added joint rotor_2_joint: type continuous, parent base_link, child rotor_2_link, origin xyz=-0.2 0.2 0.1 rpy=0 0 0, axis 0 0 1
- added joint rotor_3_joint: type continuous, parent base_link, child rotor_3_link, origin xyz=-0.2 -0.2 0.1 rpy=0 0 0, axis 0 0 1
- added joint rotor_4_joint: type continuous, parent base_link, child rotor_4_link, origin xyz=0.2 -0.2 0.1 rpy=0 0 0, axis 0 0 1
