Commit message: latest ros2_ws version

File: ros2_env/ros2_ws/src/falco_drone/urdf/sensors/quadrotor_sensors.urdf.xacro (robot description, xacro)
@@ -3,61 +3,39 @@
   <xacro:macro name="quadrotor_sensors" params="robot_name">
     <gazebo>
-      <!--
-      TODO: Convert these plugins to Ignition Gazebo compatible versions
-      <plugin name="quadrotor_imu_sim" filename="libhector_gazebo_ros_imu.so">
-        <alwaysOn>true</alwaysOn>
-        <updateRate>100.0</updateRate>
-        <bodyName>base_link</bodyName>
-        <frameId>ardrone_base_link</frameId>
-        <topicName>/${robot_name}/imu</topicName>
-        <xyzOffset>0 0 0</xyzOffset>
-	<rpyOffset>0 0 0</rpyOffset>
-        <gaussianNoise>0</gaussianNoise>
-        <accelDrift>0.5 0.5 0.5</accelDrift>
-        <accelGaussianNoise>0.35 0.35 0.3</accelGaussianNoise>
-        <rateDrift>0.0 0.0 0.0</rateDrift>
-        <rateGaussianNoise>0.00 0.00 0.00</rateGaussianNoise>
-        <headingDrift>0.0</headingDrift>
-        <headingGaussianNoise>0.00</headingGaussianNoise>
+      <!-- IMU sensor -->
+      <plugin filename="gz-sim-imu-system" name="gz::sim::systems::Imu">
+        <topic>/${robot_name}/imu</topic>
+        <enable_orientation>true</enable_orientation>
       </plugin>
-      <plugin name="quadrotor_baro_sim" filename="libhector_gazebo_ros_baro.so">
-        <alwaysOn>true</alwaysOn>
-        <updateRate>10.0</updateRate>
-        <bodyName>base_link</bodyName>
-        <topicName>/${robot_name}/pressure_height</topicName>
-        <altimeterTopicName>altimeter</altimeterTopicName>
-        <offset>0</offset>
-        <drift>0.1</drift>
-        <gaussianNoise>0.5</gaussianNoise>
+      <!-- Odometry/Ground truth -->
+      <plugin filename="gz-sim-odometry-publisher-system" name="gz::sim::systems::OdometryPublisher">
+        <odom_frame>${robot_name}/odom</odom_frame>
+        <robot_base_frame>${robot_name}/base_link</robot_base_frame>
+        <odom_topic>/${robot_name}/ground_truth/state</odom_topic>
+        <odom_publish_frequency>100</odom_publish_frequency>
       </plugin>
-      <plugin name="quadrotor_magnetic_sim" filename="libhector_gazebo_ros_magnetic.so">
-        <alwaysOn>true</alwaysOn>
-        <updateRate>10.0</updateRate>
-        <bodyName>base_link</bodyName>
-        <topicName>/${robot_name}/magnetic</topicName>
-        <offset>0 0 0</offset>
-        <drift>0.0 0.0 0.0</drift>
-        <gaussianNoise>1.3e-2 1.3e-2 1.3e-2</gaussianNoise>
-      </plugin>
-      <plugin name="quadrotor_gps_sim" filename="libhector_gazebo_ros_gps.so">
-        <alwaysOn>true</alwaysOn>
-        <updateRate>4.0</updateRate>
-        <bodyName>base_link</bodyName>
-        <topicName>/${robot_name}/fix</topicName>
-        <velocityTopicName>/${robot_name}/fix_velocity</velocityTopicName>
-        <drift>5.0 5.0 5.0</drift>
-        <gaussianNoise>0.1 0.1 0.1</gaussianNoise>
-        <velocityDrift>0 0 0</velocityDrift>
-        <velocityGaussianNoise>0.1 0.1 0.1</velocityGaussianNoise>
-      </plugin>
-      <plugin name="quadrotor_groundtruth_sim" filename="libgazebo_ros_p3d.so">
-        <alwaysOn>true</alwaysOn>
-        <updateRate>100.0</updateRate>
-        <bodyName>base_link</bodyName>
-        <topicName>/${robot_name}/ground_truth/state</topicName>
-        <gaussianNoise>0.0</gaussianNoise>
-        <frameName>map</frameName>
-      </plugin>
-      -->
+    </gazebo>
+    <!-- IMU sensor link and joint -->
+    <link name="imu_link">
+      <inertial>
+        <mass value="0.001"/>
+        <inertia ixx="0.000001" ixy="0" ixz="0" iyy="0.000001" iyz="0" izz="0.000001"/>
+      </inertial>
+    </link>
+    <joint name="imu_joint" type="fixed">
+      <parent link="base_link"/>
+      <child link="imu_link"/>
+      <origin xyz="0 0 0" rpy="0 0 0"/>
+    </joint>
+    <gazebo reference="imu_link">
+      <sensor type="imu" name="imu_sensor">
+        <always_on>1</always_on>
+        <update_rate>100</update_rate>
+        <visualize>true</visualize>
+        <plugin filename="gz-sim-imu-system" name="gz::sim::systems::Imu">
+          <topic>/${robot_name}/imu</topic>
+          <enable_orientation>true</enable_orientation>
+        </plugin>
+      </sensor>
     </gazebo>
   </xacro:macro>
